Commit message: lidar added

File: lib_robot_urdf.urdf (robot description, URDF)
Before this commit: robot lib_robot, 5 links, 4 joints
Links:
- added link lidar; visual cylinder length=0.043 radius=0.03675
- added link lidar_holder; visual cylinder length=0.012 radius=0.03925
- link base_link: geometry visual box size=0.4 0.4 0.128
Joints:
- added joint lidar_holder_joint: type fixed, parent base_link, child lidar_holder, origin xyz=-0.125 0 0.07 rpy=0 0 0
- added joint lidar_joint: type fixed, parent base_link, child lidar, origin xyz=-0.125 0 0.0973 rpy=0 0 0
